Commit message: use custom cartpole fix Warp kernel still turns white at some positions of the cartpole, ask Brennan

File: scripts/assets/cartpole_madrona.urdf (robot description, URDF)
Before this commit: robot physics, 3 links, 2 joints
Links:
- link pole: geometry collision box size=0.05 0.05 1.5; visual box size=0.05 0.05 1.5
