Commit message: remove visual shapes from URDF, to keep consistent shape count (200 instead of 400) remove debug info

File: scripts/assets/cartpole_single.urdf (robot description, URDF)
Before this commit: robot physics, 3 links, 2 joints
Links:
- link cart: geometry collision box size=0.5 0.5 0.2
- link pole: geometry collision box size=0.05 0.05 1.0
